File: hardware/Sensor-LCD5/Sensor-LCD5.kicad_sch (KiCad schematic)
At the start: 19 parts, among them Q1 TEPT5700, Q2 TEPT5700, Q3 TEPT5700, Q4 TEPT5700, Q5 TEPT5700, U1 MCP6002-xMC, U2 MCP6002-xMC, U3 MCP6002-xMC, U4 PIC32CM PL10

Commit message: work on sensor board
Parts:
- added C4: 10uF, Capacitor_SMD:C_0805_2012Metric, symbol Device:C
Connections:
- net COM: now also C4.2
- net TRACK_BLUE: now also U4.44 (ADC_1); no longer U4.47 (PWM_4)
- net TRACK_GREEN: now also U4.49 (ADC_6); no longer U4.50 (ADC_7)
- net TRACK_ORANGE: now also U4.43 (ADC_0); no longer U4.46 (PWM_3)
- net TRACK_RED: now also U4.48 (ADC_5); no longer U4.49 (ADC_6)
- net TRACK_YELLOW: now also U4.45 (ADC_2); no longer U4.48 (ADC_5)
- net VCC: now also C4.1
